File: pcb/esp8266-pcb.brd (EAGLE design)
At the start: 45.7 x 45.7 mm, 18 parts

Commit message: Added OpenHW logo.
Parts:
- added GOLD_ORB_SM1: OSHWLOGO_GOLD_ORB_LG, NBitWonder:OSHW0
Changed lines of the file:
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@@
 </element>
 <element name="T1" library="transistor" package="SOT23-BEC" value="" x="14.224" y="21.082" smashed="yes" rot="MR0">
-<attribute name="NAME" x="13.335" y="22.479" size="1.27" layer="26" font="vector" ratio="15" rot="MR0"/>
+<attribute name="NAME" x="17.907" y="21.463" size="1.27" layer="26" font="vector" ratio="15" rot="MR0"/>
 <attribute name="VALUE" x="16.129" y="17.907" size="1.27" layer="28" rot="MR0"/>
 </element>
@@
 </element>
 <element name="R2" library="rcl" package="R0805" value="12k" x="10.414" y="20.066" smashed="yes" rot="MR180">
-<attribute name="NAME" x="10.033" y="22.352" size="1.27" layer="26" font="vector" ratio="15" rot="MR180"/>
+<attribute name="NAME" x="9.779" y="22.352" size="1.27" layer="26" font="vector" ratio="15" rot="MR180"/>
 <attribute name="VALUE" x="9.779" y="22.606" size="1.27" layer="28" rot="MR180"/>
 </element>
 <element name="R3" library="rcl" package="R0805" value="12k" x="10.414" y="17.78" smashed="yes" rot="MR0">
-<attribute name="NAME" x="12.065" y="15.494" size="1.27" layer="26" font="vector" ratio="15" rot="MR0"/>
+<attribute name="NAME" x="11.811" y="15.494" size="1.27" layer="26" font="vector" ratio="15" rot="MR0"/>
 <attribute name="VALUE" x="11.049" y="15.24" size="1.27" layer="28" rot="MR0"/>
 </element>
@@
 </element>
 <element name="R5" library="rcl" package="R0805" value="10k" x="39.37" y="26.924" smashed="yes" rot="MR270">
-<attribute name="NAME" x="38.481" y="24.892" size="1.27" layer="26" font="vector" ratio="15" rot="MR180"/>
+<attribute name="NAME" x="38.735" y="24.892" size="1.27" layer="26" font="vector" ratio="15" rot="MR180"/>
 <attribute name="VALUE" x="41.91" y="27.559" size="1.27" layer="28" rot="MR270"/>
 </element>
 <element name="R6" library="rcl" package="R0805" value="10k" x="37.338" y="26.924" smashed="yes" rot="MR270">
-<attribute name="NAME" x="35.941" y="24.892" size="1.27" layer="26" font="vector" ratio="15" rot="MR180"/>
+<attribute name="NAME" x="35.687" y="24.892" size="1.27" layer="26" font="vector" ratio="15" rot="MR180"/>
 <attribute name="VALUE" x="39.878" y="27.559" size="1.27" layer="28" rot="MR270"/>
 </element>
@@
 <attribute name="VALUE" x="26.543" y="19.304" size="1.27" layer="27" ratio="10" rot="R90"/>
 </element>
+<element name="GOLD_ORB_SM1" library="NBitWonder" package="OSHW0" value="OSHWLOGO_GOLD_ORB_LG" x="24.638" y="19.05" rot="MR0"/>
 </elements>
 <signals>

Commit message: Minor board and schematic refactoring.
Parts:
- R2, R3: value 12k -> 12K
- R4: value 470 -> 470R
- R5, R6: value 10k -> 10K
Changed lines of the file:
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@@
 <attribute name="VALUE" x="8.509" y="17.907" size="1.27" layer="28" rot="MR0"/>
 </element>
-<element name="R2" library="rcl" package="R0805" value="12k" x="10.414" y="20.066" smashed="yes" rot="MR180">
+<element name="R2" library="rcl" package="R0805" value="12K" x="10.414" y="20.066" smashed="yes" rot="MR180">
 <attribute name="NAME" x="9.779" y="22.352" size="1.27" layer="26" font="vector" ratio="15" rot="MR180"/>
 <attribute name="VALUE" x="9.779" y="22.606" size="1.27" layer="28" rot="MR180"/>
 </element>
-<element name="R3" library="rcl" package="R0805" value="12k" x="10.414" y="17.78" smashed="yes" rot="MR0">
+<element name="R3" library="rcl" package="R0805" value="12K" x="10.414" y="17.78" smashed="yes" rot="MR0">
 <attribute name="NAME" x="11.811" y="15.494" size="1.27" layer="26" font="vector" ratio="15" rot="MR0"/>
 <attribute name="VALUE" x="11.049" y="15.24" size="1.27" layer="28" rot="MR0"/>
@@
 <attribute name="VALUE" x="2.286" y="9.017" size="1.27" layer="27"/>
 </element>
-<element name="R4" library="rcl" package="R0805" value="470" x="11.684" y="9.906" smashed="yes" rot="R270">
+<element name="R4" library="rcl" package="R0805" value="470R" x="11.684" y="9.906" smashed="yes" rot="R270">
 <attribute name="NAME" x="11.049" y="6.604" size="1.27" layer="25" font="vector" ratio="15"/>
 <attribute name="VALUE" x="9.144" y="10.795" size="1.27" layer="27" rot="R270"/>
 </element>
-<element name="R5" library="rcl" package="R0805" value="10k" x="39.37" y="26.924" smashed="yes" rot="MR270">
+<element name="R5" library="rcl" package="R0805" value="10K" x="39.37" y="26.924" smashed="yes" rot="MR270">
 <attribute name="NAME" x="38.735" y="24.892" size="1.27" layer="26" font="vector" ratio="15" rot="MR180"/>
 <attribute name="VALUE" x="41.91" y="27.559" size="1.27" layer="28" rot="MR270"/>
 </element>
-<element name="R6" library="rcl" package="R0805" value="10k" x="37.338" y="26.924" smashed="yes" rot="MR270">
+<element name="R6" library="rcl" package="R0805" value="10K" x="37.338" y="26.924" smashed="yes" rot="MR270">
 <attribute name="NAME" x="35.687" y="24.892" size="1.27" layer="26" font="vector" ratio="15" rot="MR180"/>
 <attribute name="VALUE" x="39.878" y="27.559" size="1.27" layer="28" rot="MR270"/>
@@
 <contactref element="C2" pad="1"/>
 <contactref element="R6" pad="2"/>
-<contactref element="R5" pad="2"/>
 <contactref element="LED1" pad="A"/>
-<wire x1="39.37" y1="25.974" x2="37.338" y2="25.974" width="0.6096" layer="16"/>
 <wire x1="37.338" y1="25.974" x2="34.986" y2="25.974" width="0.6096" layer="16"/>
 <wire x1="34.986" y1="25.974" x2="32.639" y2="28.321" width="0.6096" layer="16"/>
@@
 <via x="9.525" y="32.385" extent="1-16" drill="0.6"/>
 <wire x1="10.16" y1="26.162" x2="7.112" y2="23.114" width="0.6096" layer="1"/>
+<contactref element="R5" pad="2"/>
+<wire x1="39.37" y1="25.974" x2="37.338" y2="25.974" width="0.6096" layer="16"/>
 </signal>
 <signal name="N$3">

Commit message: Removed unused nets.
Connections:
- removed net GPIO12: MCU.14
- removed net GPIO13: MCU.15
Changed lines of the file:
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@@
 <wire x1="39.37" y1="29.591" x2="36.957" y2="32.004" width="0.4064" layer="16"/>
-</signal>
-<signal name="GPIO13">
-<contactref element="MCU" pad="15"/>
-</signal>
-<signal name="GPIO12">
-<contactref element="MCU" pad="14"/>
 </signal>
 <signal name="GPIO16">

Commit message: Minor board refactoring.
Parts:
- renumbered JP1 to PWRJACK
Changed lines of the file:
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@@
 <attribute name="VALUE" x="19.685" y="12.827" size="1.27" layer="27" ratio="10" rot="R270"/>
 </element>
-<element name="JP1" library="SparkFun-Connectors" package="POWER_JACK_PTH" value="POWER_JACKPTH" x="18.288" y="-3.302" smashed="yes">
+<element name="PWRJACK" library="SparkFun-Connectors" package="POWER_JACK_PTH" value="POWER_JACKPTH" x="18.288" y="-3.302" smashed="yes">
 <attribute name="PROD_ID" value="CONN-08197" x="62.738" y="-29.972" size="1.778" layer="27" display="off"/>
-<attribute name="NAME" x="14.478" y="1.778" size="0.4064" layer="25" font="vector" ratio="15"/>
+<attribute name="NAME" x="15.24" y="0.762" size="1.016" layer="25" font="vector" ratio="15"/>
 <attribute name="VALUE" x="14.478" y="0.508" size="0.4064" layer="27"/>
 </element>
@@
 <contactref element="PROG" pad="4"/>
 <contactref element="MCU" pad="1"/>
-<contactref element="JP1" pad="GNDBREAK"/>
-<contactref element="JP1" pad="GND"/>
+<contactref element="PWRJACK" pad="GNDBREAK"/>
+<contactref element="PWRJACK" pad="GND"/>
 <contactref element="U$2" pad="P$3"/>
 <contactref element="ICSP" pad="2"/>
@@
 </signal>
 <signal name="VIN">
-<contactref element="JP1" pad="PWR"/>
+<contactref element="PWRJACK" pad="PWR"/>
 <contactref element="U$2" pad="P$1"/>
 <contactref element="ICSP" pad="1"/>

Commit message: GPIO15 grounded with 12K resistor.
Parts:
- added R7: 12K, rcl:R0805
Connections:
- new net N$5: MCU.2, R7.1
- net GND: now also R7.2
Other:
- board text added: "IOT BAROMETER v0.1.1"
- board text removed: "IOT BAROMETER v0.1"
Changed lines of the file:
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@@
 <wire x1="45.72" y1="45.72" x2="0" y2="45.72" width="0" layer="20"/>
 <wire x1="0" y1="45.72" x2="0" y2="0" width="0" layer="20"/>
-<text x="12.446" y="44.196" size="1.4224" layer="26" font="vector" ratio="15" rot="MR180" align="center">IOT BAROMETER v0.1</text>
+<text x="12.7" y="44.196" size="1.4224" layer="26" font="vector" ratio="15" rot="MR180" align="center">IOT BAROMETER v0.1.1</text>
 <text x="12.446" y="42.418" size="1.27" layer="26" font="vector" ratio="15" rot="MR0" align="center">ivo.slanina@gmail.com</text>
 </plain>
@@
 </element>
 <element name="GOLD_ORB_SM1" library="NBitWonder" package="OSHW0" value="OSHWLOGO_GOLD_ORB_LG" x="24.638" y="19.05" rot="MR0"/>
+<element name="R7" library="rcl" package="R0805" value="12K" x="1.778" y="-7.366"/>
 </elements>
 <signals>
@@
 <via x="38.862" y="43.434" extent="1-16" drill="0.6"/>
 <via x="8.382" y="31.75" extent="1-16" drill="0.6"/>
+<contactref element="R7" pad="2"/>
+<wire x1="3.3528" y1="2.3114" x2="2.728" y2="-7.366" width="0" layer="19" extent="1-1"/>
 </signal>
 <signal name="N$1">
@@
 <wire x1="23.622" y1="18.034" x2="22.352" y2="16.764" width="0.6096" layer="16"/>
 </signal>
+<signal name="N$5">
+<contactref element="MCU" pad="2"/>
+<contactref element="R7" pad="1"/>
+<wire x1="0.828" y1="-7.366" x2="18.74" y2="25.082" width="0" layer="19" extent="1-1"/>
+</signal>
 </signals>
