File: pcb/esp8266-pcb.brd (EAGLE design)
At the start: 45.7 x 45.7 mm, 21 parts

Commit message: Added new board designs.
Parts:
- removed GOLD_ORB_SM1: OSHWLOGO_GOLD_ORB_LG, NBitWonder:OSHW0
- added C3: 100nF, rcl:C0805
- added R10, R11, R8, R9: 12K, rcl:R0805
- added U$1: OSHW-LOGOL, SparkFun:OSHW-LOGO-L
- R1: value ??R -> 82R
- moved ISPPWR 9.53 mm to (25.1, 23.9)
- moved PWR 8.32 mm to (30.7, 26.2), turned to 270 degrees
- moved C1 2.30 mm to (25.9, 15.7)
Connections:
- new net EN: ESP8266.11, R11.1
- new net GPIO13: ESP8266.15, R5.1, SENSOR_CONN.3
- net +3V3: now also R10.2, R11.2, R8.2, R9.2; no longer ESP8266.11
- net GND: now also C3.1
- net GPIO0: now also R8.1
- net GPIO2: now also R9.1; no longer R5.1, SENSOR_CONN.3
- net NRST: now also C3.2, R10.1
Routing:
- net GPIO13: track 0.00 -> 43.7 mm, vias 0 -> 2
- net GPIO2: track 26.2 -> 8.01 mm, vias 0 -> 1
- net N$6: track 11.5 -> 24.0 mm
- net VIN: track 32.7 -> 44.4 mm
- net +3V3: track 85.8 -> 76.1 mm, vias 3 -> 4
- net EN: track 0.00 -> 7.26 mm, vias 0 -> 1
- net NRST: track 18.4 -> 23.5 mm
- net GPIO0: track 29.9 -> 27.3 mm, vias 1 -> 2
- net N$2: track 23.3 -> 25.2 mm
- net GPIO14: track 42.6 -> 41.1 mm
- net DTR: track 15.6 -> 14.8 mm
Other:
- board text added: "ESP8266 NODE v0.1.2"
- board text added: "mqopen.org"
- board text removed: "ESP8266 NODE v0.1.1"
- board text removed: "ivo.slanina@gmail.com"
